File: hardware/bd950_interface/bd950_interface.sch (EAGLE design)
At the start: 34 parts, among them IC1 FT4232HL, IC2 MAX208ECWG, IC3 4050D, IC4 AT93C46A-10SQ-2.7, IC5 786TV, X1 ECG.0B.304.CLV

Commit message: WIP Fix BD950 interface board layout issues
Parts:
- removed IC5: 786TV, linear:786TV
- added IC6: LM317MDT, v-reg:LM317MDT
- added R11: 383, resistor:R-US_R0603
- added R13: 649, resistor:R-US_R0603
- U$2: value PCN13-64S-2.54DS(71) -> 294721
Connections:
- new net N$2: IC6.ADJ, R11.2, R13.2
- net +3V3: now also IC6.OUT, R13.1; no longer IC5.VO
- net GND: now also R11.1; no longer IC5.GND
- net VDD: now also IC6.IN; no longer IC5.VI
Other:
- note added: "ERNI P/N: 294721"
- note removed: "Hirose PCN13-64S-2.54DS(71)"
- moved on the sheet: C4
Changed lines of the file:
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@@
 <part name="GND38" library="supply1" deviceset="GND" device=""/>
 <part name="GND44" library="supply1" deviceset="GND" device=""/>
-<part name="U$2" library="adafruit" deviceset="TRIMBLE_BD950" device="" value="PCN13-64S-2.54DS(71)"/>
+<part name="U$2" library="adafruit" deviceset="TRIMBLE_BD950" device="" value="294721"/>
 <part name="GND3" library="supply1" deviceset="GND" device=""/>
 <part name="R1" library="rcl" deviceset="R-US_" device="R0603" value="0"/>
@@
 <part name="R3" library="rcl" deviceset="R-US_" device="R0603" value="10k"/>
 <part name="GND6" library="supply1" deviceset="GND" device=""/>
-<part name="X1" library="con-lemo" deviceset="EZG-?-304" device="0B" value="ECG.0B.304.CLV"/>
 <part name="GND7" library="supply1" deviceset="GND" device=""/>
 <part name="IC1" library="ftdichip-6" deviceset="FT4232H" device="L"/>
@@
 <part name="+3V7" library="supply1" deviceset="+3V3" device=""/>
 <part name="+3V8" library="supply1" deviceset="+3V3" device=""/>
-<part name="IC5" library="linear" deviceset="78*" device="TV" technology="6"/>
 <part name="+3V9" library="supply1" deviceset="+3V3" device=""/>
 <part name="C4" library="resistor" deviceset="C-US" device="C0805" value="10uF"/>
-<part name="GND15" library="supply1" deviceset="GND" device=""/>
 <part name="GND16" library="supply1" deviceset="GND" device=""/>
 <part name="C5" library="resistor" deviceset="C-US" device="C0805" value="10uF"/>
@@
 <part name="+3V5" library="supply1" deviceset="+3V3" device=""/>
 <part name="+3V10" library="supply1" deviceset="+3V3" device=""/>
+<part name="IC6" library="v-reg" deviceset="LM317?*" device="" technology="MDT"/>
+<part name="R11" library="resistor" deviceset="R-US_" device="R0603" value="383"/>
+<part name="R13" library="resistor" deviceset="R-US_" device="R0603" value="649"/>
+<part name="GND15" library="supply1" deviceset="GND" device=""/>
+<part name="X1" library="con-lemo" deviceset="EZG-?-304" device="0B" value="ECG.0B.304.CLV"/>
 </parts>
 <sheets>
@@
 <plain>
 <text x="121.92" y="203.2" size="3.81" layer="97">Connector</text>
-<text x="187.96" y="83.82" size="1.778" layer="97">Hirose PCN13-64S-2.54DS(71)</text>
+<text x="195.58" y="83.82" size="1.778" layer="97">ERNI P/N: 294721</text>
 </plain>
 <instances>
@@
 <instance part="R3" gate="G$1" x="38.1" y="58.42" rot="R180"/>
 <instance part="GND6" gate="1" x="60.96" y="48.26"/>
-<instance part="X1" gate="G$1" x="50.8" y="129.54" rot="R180"/>
 <instance part="GND7" gate="1" x="58.42" y="124.46"/>
 <instance part="IC3" gate="A" x="124.46" y="78.74"/>
@@
 <instance part="IC3" gate="P" x="172.72" y="60.96"/>
 <instance part="+3V10" gate="G$1" x="172.72" y="73.66"/>
+<instance part="X1" gate="G$1" x="50.8" y="129.54" rot="R180"/>
 </instances>
 <busses>
@@
 </segment>
 <segment>
-<pinref part="X1" gate="G$1" pin="1"/>
 <pinref part="GND7" gate="1" pin="GND"/>
 <wire x1="55.88" y1="129.54" x2="58.42" y2="129.54" width="0.1524" layer="91"/>
 <wire x1="58.42" y1="129.54" x2="58.42" y2="127" width="0.1524" layer="91"/>
-<pinref part="X1" gate="G$1" pin="4"/>
 <wire x1="55.88" y1="137.16" x2="58.42" y2="137.16" width="0.1524" layer="91"/>
 <wire x1="58.42" y1="137.16" x2="58.42" y2="129.54" width="0.1524" layer="91"/>
 <junction x="58.42" y="129.54"/>
+<pinref part="X1" gate="G$1" pin="1"/>
+<pinref part="X1" gate="G$1" pin="4"/>
 </segment>
 <segment>
@@
 <net name="1PPS_EXT0" class="0">
 <segment>
-<pinref part="X1" gate="G$1" pin="3"/>
 <wire x1="55.88" y1="134.62" x2="91.44" y2="134.62" width="0.1524" layer="91"/>
 <label x="91.44" y="134.62" size="1.778" layer="95" rot="MR0"/>
+<pinref part="X1" gate="G$1" pin="3"/>
 </segment>
 <segment>
@@
 <net name="1PPS_EXT1" class="0">
 <segment>
-<pinref part="X1" gate="G$1" pin="2"/>
 <wire x1="55.88" y1="132.08" x2="91.44" y2="132.08" width="0.1524" layer="91"/>
 <label x="91.44" y="132.08" size="1.778" layer="95" rot="MR0"/>
+<pinref part="X1" gate="G$1" pin="2"/>
 </segment>
 <segment>
@@
 <instance part="+3V7" gate="G$1" x="96.52" y="182.88"/>
 <instance part="+3V8" gate="G$1" x="76.2" y="193.04"/>
-<instance part="IC5" gate="A1" x="210.82" y="193.04"/>
 <instance part="+3V9" gate="G$1" x="228.6" y="203.2"/>
-<instance part="C4" gate="G$1" x="228.6" y="187.96"/>
-<instance part="GND15" gate="1" x="210.82" y="180.34"/>
-<instance part="GND16" gate="1" x="228.6" y="180.34"/>
+<instance part="C4" gate="G$1" x="228.6" y="177.8"/>
+<instance part="GND16" gate="1" x="228.6" y="167.64"/>
 <instance part="C5" gate="G$1" x="193.04" y="187.96"/>
 <instance part="GND17" gate="1" x="193.04" y="180.34"/>
@@
 <instance part="C10" gate="G$1" x="233.68" y="154.94" rot="R90"/>
 <instance part="+3V5" gate="G$1" x="251.46" y="165.1"/>
+<instance part="IC6" gate="G$1" x="210.82" y="198.12"/>
+<instance part="R11" gate="G$1" x="210.82" y="175.26" rot="R90"/>
+<instance part="R13" gate="G$1" x="218.44" y="182.88" rot="R180"/>
+<instance part="GND15" gate="1" x="210.82" y="167.64"/>
 </instances>
 <busses>
@@
 <pinref part="C4" gate="G$1" pin="2"/>
 <pinref part="GND16" gate="1" pin="GND"/>
+<wire x1="228.6" y1="170.18" x2="228.6" y2="172.72" width="0.1524" layer="91"/>
 </segment>
 <segment>
 <pinref part="C5" gate="G$1" pin="2"/>
 <pinref part="GND17" gate="1" pin="GND"/>
-</segment>
-<segment>
-<pinref part="GND15" gate="1" pin="GND"/>
-<pinref part="IC5" gate="A1" pin="GND"/>
-<wire x1="210.82" y1="182.88" x2="210.82" y2="185.42" width="0.1524" layer="91"/>
 </segment>
 <segment>
@@
 <pinref part="IC2" gate="P" pin="GND"/>
 <junction x="251.46" y="139.7"/>
+</segment>
+<segment>
+<pinref part="R11" gate="G$1" pin="1"/>
+<pinref part="GND15" gate="1" pin="GND"/>
 </segment>
 </net>
@@
 </segment>
 <segment>
-<pinref part="IC5" gate="A1" pin="VO"/>
 <pinref part="+3V9" gate="G$1" pin="+3V3"/>
-<wire x1="220.98" y1="193.04" x2="228.6" y2="193.04" width="0.1524" layer="91"/>
-<wire x1="228.6" y1="193.04" x2="228.6" y2="200.66" width="0.1524" layer="91"/>
+<wire x1="218.44" y1="198.12" x2="228.6" y2="198.12" width="0.1524" layer="91"/>
+<wire x1="228.6" y1="198.12" x2="228.6" y2="200.66" width="0.1524" layer="91"/>
 <pinref part="C4" gate="G$1" pin="1"/>
-<wire x1="228.6" y1="190.5" x2="228.6" y2="193.04" width="0.1524" layer="91"/>
-<junction x="228.6" y="193.04"/>
+<wire x1="228.6" y1="180.34" x2="228.6" y2="182.88" width="0.1524" layer="91"/>
+<junction x="228.6" y="198.12"/>
+<pinref part="IC6" gate="G$1" pin="OUT"/>
+<pinref part="R13" gate="G$1" pin="1"/>
+<wire x1="228.6" y1="182.88" x2="228.6" y2="198.12" width="0.1524" layer="91"/>
+<wire x1="223.52" y1="182.88" x2="228.6" y2="182.88" width="0.1524" layer="91"/>
+<junction x="228.6" y="182.88"/>
 </segment>
 <segment>
@@
 <segment>
 <pinref part="C5" gate="G$1" pin="1"/>
-<wire x1="193.04" y1="200.66" x2="193.04" y2="193.04" width="0.1524" layer="91"/>
-<pinref part="IC5" gate="A1" pin="VI"/>
-<wire x1="193.04" y1="193.04" x2="193.04" y2="190.5" width="0.1524" layer="91"/>
-<wire x1="200.66" y1="193.04" x2="193.04" y2="193.04" width="0.1524" layer="91"/>
-<junction x="193.04" y="193.04"/>
+<wire x1="193.04" y1="200.66" x2="193.04" y2="198.12" width="0.1524" layer="91"/>
+<wire x1="193.04" y1="198.12" x2="193.04" y2="190.5" width="0.1524" layer="91"/>
+<wire x1="203.2" y1="198.12" x2="193.04" y2="198.12" width="0.1524" layer="91"/>
+<junction x="193.04" y="198.12"/>
 <pinref part="VDD4" gate="G$1" pin="VDD"/>
-</segment>
-</net>
+<pinref part="IC6" gate="G$1" pin="IN"/>
+</segment>
+</net>
+<net name="N$2" class="0">
+<segment>
+<pinref part="IC6" gate="G$1" pin="ADJ"/>
+<pinref part="R11" gate="G$1" pin="2"/>
+<wire x1="210.82" y1="190.5" x2="210.82" y2="182.88" width="0.1524" layer="91"/>
+<pinref part="R13" gate="G$1" pin="2"/>
+<wire x1="210.82" y1="182.88" x2="210.82" y2="180.34" width="0.1524" layer="91"/>
+<wire x1="213.36" y1="182.88" x2="210.82" y2="182.88" width="0.1524" layer="91"/>
+<junction x="210.82" y="182.88"/>
+</segment>
+</net>

Commit message: Rev 2 of BD950 interface board
Parts:
- removed X1: ECG.0B.304.CLV, con-lemo:EZG-0B-304
- added C11: 0.1uF, resistor:C-USC0603
- added R14: 10k, rcl:R-US_R0603
- added U$3: ECG.0B.304.CLV, adafruit:ECG.0B.CLV
- added U$4: SN74LVC1G123, adafruit:SN74LVC1G123
Connections:
- new net N$13: R4.1, R5.1, U$4.B
- new net N$21: C11.2, U$4.CEXT
- new net N$23: C11.1, R14.2, U$4.REXT
- net +3V3: now also R14.1, U$4./CLR, U$4.VCC
- net 1PPS_EXT0: now also U$3.3; no longer X1.3
- net 1PPS_EXT1: now also U$3.2; no longer X1.2
- net GND: now also U$3.1, U$3.4, U$4./A, U$4.GND; no longer X1.1, X1.4
- net N$8: now also U$4.Q; no longer R4.1, R5.1
Other:
- note added: "1PPS from receiver is ~7us wide. R=10k, C=0.1uF makes it ~1ms wide."
- note added: "Designed to fit with the BD950 in a Hammond 1457L1202BK"
- moved on the sheet: C7, LED1, LED2, LED3, R1, R19, R2, R3, R4, R5, U$1
